Commit message: small fixes

File: onrobot_rg2_description/urdf/onrobot_rg2.urdf.xacro (robot description, xacro)
@@ -34,5 +34,7 @@
   </xacro:macro>
   <xacro:macro name="onrobot_rg2"
-    params="parent_link xyz rpy">
+    params="parent_link
+            xyz rpy
+            use_ros_control:=True">
     <joint name="parent_to_base_fixed_joint" type="fixed">
       <parent link="${parent_link}" />
@@ -50,11 +52,11 @@
         <origin xyz="0.0 0.0 0.0" rpy="0.0 0.0 0.0" />
         <geometry>
-          <mesh filename="file://$(find ur_components_description)/meshes/hand.stl" />
-        </geometry>
-      </collision>
-      <visual>
-        <origin xyz="0.0 0.0 0.0" rpy="0.0 0.0 0.0" />
-        <geometry>
-          <mesh filename="file://$(find ur_components_description)/meshes/hand.dae" />
+          <mesh filename="file://$(find onrobot_rg2_description)/meshes/hand.stl" />
+        </geometry>
+      </collision>
+      <visual>
+        <origin xyz="0.0 0.0 0.0" rpy="0.0 0.0 0.0" />
+        <geometry>
+          <mesh filename="file://$(find onrobot_rg2_description)/meshes/hand.dae" />
         </geometry>
       </visual>
@@ -81,11 +83,11 @@
         <origin xyz="0.0 0.0 0.0" rpy="0.0 0.0 0.0" />
         <geometry>
-          <mesh filename="file://$(find ur_components_description)/meshes/moment_arm.stl" />
-        </geometry>
-      </collision>
-      <visual>
-        <origin xyz="0.0 0.0 0.0" rpy="0.0 0.0 0.0" />
-        <geometry>
-          <mesh filename="file://$(find ur_components_description)/meshes/moment_arm.dae" />
+          <mesh filename="file://$(find onrobot_rg2_description)/meshes/moment_arm.stl" />
+        </geometry>
+      </collision>
+      <visual>
+        <origin xyz="0.0 0.0 0.0" rpy="0.0 0.0 0.0" />
+        <geometry>
+          <mesh filename="file://$(find onrobot_rg2_description)/meshes/moment_arm.dae" />
         </geometry>
       </visual>
@@ -118,11 +120,11 @@
         <origin xyz="0.0 0.0 0.0" rpy="0.0 0.0 0.0" />
         <geometry>
-          <mesh filename="file://$(find ur_components_description)/meshes/finger.stl" />
-        </geometry>
-      </collision>
-      <visual>
-        <origin xyz="0.0 0.0 0.0" rpy="0.0 0.0 0.0" />
-        <geometry>
-          <mesh filename="file://$(find ur_components_description)/meshes/finger.dae" />
+          <mesh filename="file://$(find onrobot_rg2_description)/meshes/finger.stl" />
+        </geometry>
+      </collision>
+      <visual>
+        <origin xyz="0.0 0.0 0.0" rpy="0.0 0.0 0.0" />
+        <geometry>
+          <mesh filename="file://$(find onrobot_rg2_description)/meshes/finger.dae" />
         </geometry>
       </visual>
@@ -155,11 +157,11 @@
         <origin xyz="0.0 0.0 0.0" rpy="0.0 0.0 0.0" />
         <geometry>
-          <mesh filename="file://$(find ur_components_description)/meshes/truss_arm.stl" />
-        </geometry>
-      </collision>
-      <visual>
-        <origin xyz="0.0 0.0 0.0" rpy="0.0 0.0 0.0" />
-        <geometry>
-          <mesh filename="file://$(find ur_components_description)/meshes/truss_arm.dae" />
+          <mesh filename="file://$(find onrobot_rg2_description)/meshes/truss_arm.stl" />
+        </geometry>
+      </collision>
+      <visual>
+        <origin xyz="0.0 0.0 0.0" rpy="0.0 0.0 0.0" />
+        <geometry>
+          <mesh filename="file://$(find onrobot_rg2_description)/meshes/truss_arm.dae" />
         </geometry>
       </visual>
@@ -192,11 +194,11 @@
         <origin xyz="0.0 0.0 -0.02" rpy="${pi} 0.0 0.0" />
         <geometry>
-          <mesh filename="file://$(find ur_components_description)/meshes/moment_arm.stl" />
-        </geometry>
-      </collision>
-      <visual>
-        <origin xyz="0.0 0.0 -0.02" rpy="${pi} 0.0 0.0" />
-        <geometry>
-          <mesh filename="file://$(find ur_components_description)/meshes/moment_arm.dae" />
+          <mesh filename="file://$(find onrobot_rg2_description)/meshes/moment_arm.stl" />
+        </geometry>
+      </collision>
+      <visual>
+        <origin xyz="0.0 0.0 -0.02" rpy="${pi} 0.0 0.0" />
+        <geometry>
+          <mesh filename="file://$(find onrobot_rg2_description)/meshes/moment_arm.dae" />
         </geometry>
       </visual>
@@ -229,11 +231,11 @@
         <origin xyz="0.0 0.0 -0.02" rpy="${pi} 0.0 0.0" />
         <geometry>
-          <mesh filename="file://$(find ur_components_description)/meshes/finger.stl" />
-        </geometry>
-      </collision>
-      <visual>
-        <origin xyz="0.0 0.0 -0.02" rpy="${pi} 0.0 0.0" />
-        <geometry>
-          <mesh filename="file://$(find ur_components_description)/meshes/finger.dae" />
+          <mesh filename="file://$(find onrobot_rg2_description)/meshes/finger.stl" />
+        </geometry>
+      </collision>
+      <visual>
+        <origin xyz="0.0 0.0 -0.02" rpy="${pi} 0.0 0.0" />
+        <geometry>
+          <mesh filename="file://$(find onrobot_rg2_description)/meshes/finger.dae" />
         </geometry>
       </visual>
@@ -266,11 +268,11 @@
         <origin xyz="0.0 0.0 -0.02" rpy="${pi} 0.0 0.0" />
         <geometry>
-          <mesh filename="file://$(find ur_components_description)/meshes/truss_arm.stl" />
-        </geometry>
-      </collision>
-      <visual>
-        <origin xyz="0.0 0.0 -0.02" rpy="${pi} 0.0 0.0" />
-        <geometry>
-          <mesh filename="file://$(find ur_components_description)/meshes/truss_arm.dae" />
+          <mesh filename="file://$(find onrobot_rg2_description)/meshes/truss_arm.stl" />
+        </geometry>
+      </collision>
+      <visual>
+        <origin xyz="0.0 0.0 -0.02" rpy="${pi} 0.0 0.0" />
+        <geometry>
+          <mesh filename="file://$(find onrobot_rg2_description)/meshes/truss_arm.dae" />
         </geometry>
       </visual>
@@ -283,10 +285,10 @@
       </inertial>
     </link>
-    <!-- <gazebo>
-      <plugin name="gazebo_ros_control" filename="libgazebo_ros_control.so">
-        <robotNamespace>/rg2</robotNamespace>
-        <robotSimType>gazebo_ros_control/DefaultRobotHWSim</robotSimType>
-      </plugin>
-    </gazebo> -->
+    <xacro:if value="${use_ros_control}">
+      <gazebo>
+        <plugin name="gazebo_ros_control" filename="libgazebo_ros_control.so">
+        </plugin>
+      </gazebo>
+    </xacro:if>
   </xacro:macro>
 </robot>

Commit message: fix launches and urdf

File: onrobot_rg2_description/urdf/onrobot_rg2.urdf.xacro (robot description, xacro)
@@ -74,5 +74,5 @@
       <origin xyz="0.105 0.017 0.010" rpy="0.0 0.0 0.0" />
       <axis xyz="0.0 0.0 1.0" />
-      <limit velocity="3.14" effort="10.6" lower="${-0.45}" upper="${pi*0.5}" />
+      <limit velocity="3.14" effort="10.6" lower="${-0.45}" upper="${1.0}" />
       <dynamics damping="0.1" friction="0.0" />
       <implicitSpringDamper>True</implicitSpringDamper>
